File: hardware/Qlock250mm/pcb/Qlock250mm/Qlock250mm.kicad_pcb (KiCad board)
At the start: 2 copper layers, 240 x 240 mm, 232 parts, among them U1 XIAO-ESP32-S3-Plus-SMD, U2 74AHCT1G125

Commit message: Update the clock enclosure and PCB design
Parts:
- added C116: 1uF, Capacitor_SMD:C_0603_1608Metric, F.Cu at (160.0, 56.0)
- added C117: 1000uF, Capacitor_SMD:CP_Elec_10x10, F.Cu at (243.3, 260.8)
- added R2: 1k5, Resistor_SMD:R_0402_1005Metric, F.Cu at (160.3, 54.4)
- added R3: 1k5, Resistor_SMD:R_0402_1005Metric, F.Cu at (160.4, 61.8)
- added U3: TSL25911FN, OptoDevice:AMS_TSL25911FN, F.Cu at (160.0, 59.2)
- C115, R1, U2: moved to F.Cu
- moved R1 94.4 mm to (230.2, 261.8), turned to 180 degrees
- moved U2 87.0 mm to (226.7, 260.8), turned to 0 degrees
- moved C115 86.4 mm to (226.3, 257.8), turned to 180 degrees
Connections:
- net Net-(U1-D3) renamed /LED_Data_3V3
- U1 pad 12: unconnected-(U1-3V3_OUT-Pad12) -> +3.3V
- U1 pad 13: unconnected-(U1-GND-Pad13) -> GND
- U1 pad 14: unconnected-(U1-VBUS-Pad14) -> +5V
- U1 pad 5: unconnected-(U1-D4-Pad5) -> I2C_SDA
- U1 pad 6: unconnected-(U1-D5-Pad6) -> I2C_SCL
Routing:
- net +3.3V: track 0.00 -> 199.2 mm, vias 0 -> 2
- net I2C_SDA: track 0.00 -> 195.7 mm, vias 0 -> 1
- net I2C_SCL: track 0.00 -> 190.2 mm, vias 0 -> 2
- net Net-(D1-DIN): track 122.1 -> 37.7 mm, vias 1 -> 2
- net /LED_Data_3V3: track 10.2 -> 85.5 mm, vias 0 -> 1
- net +5V: track 51.3 -> 86.4 mm, vias 24 -> 26
- net GND: track 32.9 -> 64.2 mm
Other:
- outline, holes or cut-outs redrawn
