File: hardware/Qlock250mm/pcb/Qlock250mm/Qlock250mm.kicad_sch (KiCad schematic)
At the start: 232 parts, among them U1 XIAO-ESP32-S3-Plus-SMD, U2 74AHCT1G125

Commit message: Update the clock enclosure and PCB design
Parts:
- added C116: 1uF, Capacitor_SMD:C_0603_1608Metric, symbol Device:C_Polarized_Small
- added C117: 1000uF, Capacitor_SMD:CP_Elec_10x10, symbol Device:C_Polarized_Small
- added R2, R3: 1k5, Resistor_SMD:R_0402_1005Metric, symbol Device:R
- added U3: TSL25911FN, OptoDevice:AMS_TSL25911FN, symbol Sensor_Optical:TSL25911FN
- C1, C10, C100, C101, C102, C103, C104, C105, C106, C107, C108, C109, C11, C110, C111, C112, C113, C114, C115, C12, C13, C14, C15, C16, C17, C18, C19, C2, C20, C21, C22, C23, C24, C25, C26, C27, C28, C29, C3, C30, C31, C32, C33, C34, C35, C36, C37, C38, C39, C4, C40, C41, C42, C43, C44, C45, C46, C47, C48, C49, C5, C50, C51, C52, C53, C54, C55, C56, C57, C58, C59, C6, C60, C61, C62, C63, C64, C65, C66, C67, C68, C69, C7, C70, C71, C72, C73, C74, C75, C76, C77, C78, C79, C8, C80, C81, C82, C83, C84, C85, C86, C87, C88, C89, C9, C90, C91, C92, C93, C94, C95, C96, C97, C98, C99: LCSC Part # (none) -> C1588
- D1, D10, D100, D101, D102, D103, D104, D105, D106, D107, D108, D109, D11, D110, D111, D112, D113, D114, D12, D13, D14, D15, D16, D17, D18, D19, D2, D20, D21, D22, D23, D24, D25, D26, D27, D28, D29, D3, D30, D31, D32, D33, D35, D36, D37, D38, D39, D4, D40, D41, D42, D43, D44, D45, D46, D47, D48, D49, D5, D50, D51, D52, D53, D54, D55, D56, D57, D58, D59, D6, D60, D61, D62, D63, D64, D65, D66, D67, D68, D69, D7, D70, D71, D72, D73, D74, D75, D76, D77, D78, D79, D8, D80, D81, D82, D83, D84, D85, D86, D87, D88, D89, D9, D90, D91, D92, D93, D94, D95, D96, D97, D98, D99: FT Rotation Offset (none) -> -90; LCSC Part # (none) -> C2843785
- D34: FT Rotation Offset (none) -> -90; JLCPCB Rotation Offset (none) -> -90; LCSC Part # (none) -> C2843785
- R1: LCSC Part # (none) -> C25104
- U1: now left out of the parts list
- U2: LCSC Part # (none) -> C7484
Connections:
- net +5V: now also U1.14 (VBUS), C117.1
- net GND: now also U1.13 (GND), C116.2, C117.2, U3.3 (GND)
- net +3.3V: now reaches U1.12 (3V3_OUT)
- net +3.3V: now also C116.1, R2.1, R3.1, U3.5 (VDD)
- net LED_Data_3V3: now reaches U1.4 (D3), U2.2
- net I2C_SDA: now reaches U1.5 (D4)
- net I2C_SDA: now also R2.2, U3.6 (SDA)
- net I2C_SCL: now reaches U1.6 (D5)
- net I2C_SCL: now also R3.2, U3.1 (SCL)
